File: hardware/audio-switch.sch (KiCad schematic (older format))
At the start: 15 parts, among them J1 programming conn, J8 5V connector, SW1 SW_Push, U1 ATtiny2313A-PU

Commit message: refactoring
Parts:
- removed R1, R3: 47K, Resistor_THT:R_Axial_DIN0207_L6.3mm_D2.5mm_P7.62mm_Horizontal, symbol Device:R_Small
- added D4: LED, LED_THT:LED_D3.0mm, symbol Device:LED
- renumbered D4 to D1, D3 to D2, D2 to D3, D1 to D5, D0-1 to D6, J8 to J1, J1 to J2, R2 to R1, R4 to R2
Connections:
- net at SW1.1: now also U1.11 (PD6); no longer U1.9 (PD5)
- net at D1.1 (K), D2.1 (K), D3.1 (K)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: now also D4.1 (K)
- net at U1.5 (PA0/XTAL1): now also D4.2 (A)
- new net audio_5: U1.9 (PD5)
Other:
- moved on the sheet: R2
Changed lines of the file:
@@
 EESchema Schematic File Version 4
-LIBS:audio-line-selector-cache
+LIBS:audio-switch-cache
 EELAYER 26 0
 EELAYER END
@@
 encoding utf-8
 Sheet 1 2
-Title "Audio line selector"
+Title "Audio switch"
 Date "2021-06-27"
 Rev "v1.0"
@@
 $EndComp
 $Comp
-L Device:R R4
+L Device:R R2
 U 1 1 60BB4CA6
-P 5650 2100
-F 0 "R4" V 5443 2100 50  0000 C CNN
-F 1 "270R" V 5534 2100 50  0000 C CNN
-F 2 "Resistor_THT:R_Axial_DIN0207_L6.3mm_D2.5mm_P7.62mm_Horizontal" V 5580 2100 50  0001 C CNN
-F 3 "~" H 5650 2100 50  0001 C CNN
-	1    5650 2100
+P 5650 1900
+F 0 "R2" V 5443 1900 50  0000 C CNN
+F 1 "270R" V 5534 1900 50  0000 C CNN
+F 2 "Resistor_THT:R_Axial_DIN0207_L6.3mm_D2.5mm_P7.62mm_Horizontal" V 5580 1900 50  0001 C CNN
+F 3 "~" H 5650 1900 50  0001 C CNN
+	1    5650 1900
 	0    1    1    0
 $EndComp
 $Comp
-L Device:LED D1
+L Device:LED D5
 U 1 1 60BB55B4
 P 5150 2200
-F 0 "D1" H 5142 1945 50  0001 C CNN
+F 0 "D5" H 4850 2200 50  0000 C CNN
 F 1 "LED" H 5142 2036 50  0001 C CNN
 F 2 "LED_THT:LED_D3.0mm" H 5150 2200 50  0001 C CNN
@@
 $EndComp
 $Comp
-L Device:LED D0-1
+L Device:LED D6
 U 1 1 60BB584C
 P 5150 2100
-F 0 "D0-1" H 5142 1845 50  0000 C CNN
-F 1 "LED" H 5142 1936 50  0000 C CNN
+F 0 "D6" H 4850 2100 50  0000 C CNN
+F 1 "LED" H 5142 1936 50  0001 C CNN
 F 2 "LED_THT:LED_D3.0mm" H 5150 2100 50  0001 C CNN
 F 3 "~" H 5150 2100 50  0001 C CNN
@@
 $EndComp
 $Comp
-L Device:LED D2
+L Device:LED D3
 U 1 1 60BB5A4E
 P 5150 2300
-F 0 "D2" H 5142 2045 50  0001 C CNN
+F 0 "D3" H 4850 2300 50  0000 C CNN
 F 1 "LED" H 5142 2136 50  0001 C CNN
 F 2 "LED_THT:LED_D3.0mm" H 5150 2300 50  0001 C CNN
@@
 $EndComp
 $Comp
-L Device:LED D3
+L Device:LED D2
 U 1 1 60BB5A93
 P 5150 2400
-F 0 "D3" H 5142 2145 50  0001 C CNN
+F 0 "D2" H 4850 2400 50  0000 C CNN
 F 1 "LED" H 5142 2236 50  0001 C CNN
 F 2 "LED_THT:LED_D3.0mm" H 5150 2400 50  0001 C CNN
@@
 $EndComp
 $Comp
-L Device:LED D4
+L Device:LED D1
 U 1 1 60BB5ACB
 P 5150 2500
-F 0 "D4" H 5142 2245 50  0001 C CNN
+F 0 "D1" H 4850 2500 50  0000 C CNN
 F 1 "LED" H 5142 2336 50  0001 C CNN
 F 2 "LED_THT:LED_D3.0mm" H 5150 2500 50  0001 C CNN
@@
 	4700 2500 5000 2500
 Wire Wire Line
-	5300 2100 5300 2200
-Wire Wire Line
-	5300 2200 5300 2300
-Connection ~ 5300 2200
-Wire Wire Line
 	5300 2300 5300 2400
 Connection ~ 5300 2300
@@
 	2500 6400 3100 6400
 $Comp
-L power:GND #PWR04
+L power:GND #PWR05
 U 1 1 60BDAA33
 P 2500 6400
-F 0 "#PWR04" H 2500 6150 50  0001 C CNN
+F 0 "#PWR05" H 2500 6150 50  0001 C CNN
 F 1 "GND" H 2505 6227 50  0000 C CNN
 F 2 "" H 2500 6400 50  0001 C CNN
@@
 	3250 2850 3250 4000
 $Comp
-L Connector:AVR-ISP-10 J1
+L Connector:AVR-ISP-10 J2
 U 1 1 60D2C62A
 P 1650 3000
-F 0 "J1" H 1370 3096 50  0000 R CNN
+F 0 "J2" H 1370 3096 50  0000 R CNN
 F 1 "programming conn" H 1370 3005 50  0000 R CNN
 F 2 "Connector_PinHeader_2.54mm:PinHeader_2x05_P2.54mm_Vertical" H 1650 3000 50  0001 C CNN
@@
 $EndComp
 $Comp
-L power:GND #PWR03
+L power:GND #PWR04
 U 1 1 60D2E288
 P 1550 3650
-F 0 "#PWR03" H 1550 3400 50  0001 C CNN
+F 0 "#PWR04" H 1550 3400 50  0001 C CNN
 F 1 "GND" H 1555 3477 50  0000 C CNN
 F 2 "" H 1550 3650 50  0001 C CNN
@@
 $EndComp
 $Comp
-L power:GND #PWR02
+L power:GND #PWR03
 U 1 1 60D75D9D
 P 1250 1500
-F 0 "#PWR02" H 1250 1250 50  0001 C CNN
+F 0 "#PWR03" H 1250 1250 50  0001 C CNN
 F 1 "GND" H 1255 1327 50  0000 C CNN
 F 2 "" H 1250 1500 50  0001 C CNN
@@
 	1550 1200 2250 1200
 Wire Wire Line
-	4100 6400 4750 6400
-Wire Wire Line
-	4700 3500 4850 3500
-Wire Wire Line
-	4700 3600 4750 3600
-Wire Wire Line
-	4750 3600 4750 5500
-$Comp
-L Device:R_Small R3
-U 1 1 60D9CE20
-P 4750 5600
-F 0 "R3" H 4600 5600 50  0000 L CNN
-F 1 "47K" H 4550 5500 50  0000 L CNN
-F 2 "Resistor_THT:R_Axial_DIN0207_L6.3mm_D2.5mm_P7.62mm_Horizontal" H 4750 5600 50  0001 C CNN
-F 3 "~" H 4750 5600 50  0001 C CNN
-	1    4750 5600
-	1    0    0    -1
-$EndComp
-Wire Wire Line
-	4750 5700 4750 6400
-Connection ~ 4750 6400
-Wire Wire Line
-	4750 6400 4850 6400
-Wire Wire Line
 	4850 5550 4850 6400
-Wire Wire Line
-	4850 3500 4850 5150
 $Comp
 L power:VCC #PWR01
@@
 sck
 Wire Wire Line
-	5300 2100 5500 2100
-Connection ~ 5300 2100
+	5300 1900 5500 1900
 $Comp
 L power:GND #PWR07
 U 1 1 60E010A1
-P 5800 2250
-F 0 "#PWR07" H 5800 2000 50  0001 C CNN
-F 1 "GND" H 5805 2077 50  0000 C CNN
-F 2 "" H 5800 2250 50  0001 C CNN
-F 3 "" H 5800 2250 50  0001 C CNN
-	1    5800 2250
-	1    0    0    -1
-$EndComp
-Wire Wire Line
-	5800 2100 5800 2250
+P 5800 2050
+F 0 "#PWR07" H 5800 1800 50  0001 C CNN
+F 1 "GND" H 5805 1877 50  0000 C CNN
+F 2 "" H 5800 2050 50  0001 C CNN
+F 3 "" H 5800 2050 50  0001 C CNN
+	1    5800 2050
+	1    0    0    -1
+$EndComp
+Wire Wire Line
+	5800 1900 5800 2050
 $Comp
 L power:PWR_FLAG #FLG01
@@
 Connection ~ 4100 1800
 Wire Wire Line
-	3500 2300 2550 2300
-Wire Wire Line
-	2550 2300 2550 2600
-Wire Wire Line
 	3500 2500 2850 2500
 Wire Wire Line
 	2850 2500 2850 2600
 $Comp
-L Device:R_Small R2
+L Device:R_Small R1
 U 1 1 60D797B2
 P 2850 2700
-F 0 "R2" H 2700 2700 50  0000 L CNN
+F 0 "R1" H 2700 2700 50  0000 L CNN
 F 1 "47K" H 2650 2600 50  0000 L CNN
 F 2 "Resistor_THT:R_Axial_DIN0207_L6.3mm_D2.5mm_P7.62mm_Horizontal" H 2850 2700 50  0001 C CNN
 F 3 "~" H 2850 2700 50  0001 C CNN
 	1    2850 2700
-	1    0    0    -1
-$EndComp
-$Comp
-L Device:R_Small R1
-U 1 1 60D798A6
-P 2550 2700
-F 0 "R1" H 2400 2700 50  0000 L CNN
-F 1 "47K" H 2350 2600 50  0000 L CNN
-F 2 "Resistor_THT:R_Axial_DIN0207_L6.3mm_D2.5mm_P7.62mm_Horizontal" H 2550 2700 50  0001 C CNN
-F 3 "~" H 2550 2700 50  0001 C CNN
-	1    2550 2700
 	1    0    0    -1
 $EndComp
@@
 $EndComp
 $Comp
-L power:GND #PWR05
-U 1 1 60D79954
-P 2550 2800
-F 0 "#PWR05" H 2550 2550 50  0001 C CNN
-F 1 "GND" H 2555 2627 50  0000 C CNN
-F 2 "" H 2550 2800 50  0001 C CNN
-F 3 "" H 2550 2800 50  0001 C CNN
-	1    2550 2800
-	1    0    0    -1
-$EndComp
-$Comp
-L Connector:Conn_01x02_Female J8
+L Connector:Conn_01x02_Female J1
 U 1 1 60E0DDB6
 P 1050 650
-F 0 "J8" V 990 698 50  0000 L CNN
+F 0 "J1" V 990 698 50  0000 L CNN
 F 1 "5V connector" V 899 698 50  0000 L CNN
 F 2 "Connector_Wire:SolderWirePad_1x02_P3.81mm_Drill1mm" H 1050 650 50  0001 C CNN
@@
 	1050 850  1050 1200
 $Comp
-L power:GND #PWR037
+L power:GND #PWR02
 U 1 1 60E10DFB
 P 950 850
-F 0 "#PWR037" H 950 600 50  0001 C CNN
+F 0 "#PWR02" H 950 600 50  0001 C CNN
 F 1 "GND" H 955 677 50  0000 C CNN
 F 2 "" H 950 850 50  0001 C CNN
@@
 	650  1200 1050 1200
 Connection ~ 1050 1200
+Wire Wire Line
+	4100 6400 4850 6400
+Wire Wire Line
+	4700 3600 4850 3600
+Wire Wire Line
+	4850 3600 4850 5150
+Text GLabel 4700 3500 2    50   Output ~ 0
+audio_5
+$Comp
+L Device:LED D4
+U 1 1 60E3A861
+P 5150 1650
+F 0 "D4" H 4850 1650 50  0000 C CNN
+F 1 "LED" H 5142 1486 50  0001 C CNN
+F 2 "LED_THT:LED_D3.0mm" H 5150 1650 50  0001 C CNN
+F 3 "~" H 5150 1650 50  0001 C CNN
+	1    5150 1650
+	-1   0    0    1
+$EndComp
+Wire Wire Line
+	3500 2300 3000 2300
+Wire Wire Line
+	3000 2300 3000 1650
+Wire Wire Line
+	3000 1650 5000 1650
+Wire Wire Line
+	5300 1650 5300 1900
+Connection ~ 5300 2200
+Wire Wire Line
+	5300 2200 5300 2300
+Connection ~ 5300 2100
+Wire Wire Line
+	5300 2100 5300 2200
+Connection ~ 5300 1900
+Wire Wire Line
+	5300 1900 5300 2100
 $EndSCHEMATC
