File: hardware/file60E4F6C9.sch (KiCad schematic (older format))
At the start: 55 parts

Commit message: refactoring
Parts:
- removed C?: 10uF, Capacitor_SMD:CP_Elec_3x5.3, symbol Device:CP1
- removed C?: 10uF, Capacitor_SMD:CP_Elec_3x5.4, symbol Device:CP1
- removed J?: AudioJack3, Connector_Audio:Jack_3.5mm_CUI_SJ1-3533NG_Horizontal, symbol Connector:AudioJack3
- removed R? (x4): 47K, Resistor_SMD:R_0201_0603Metric, symbol Device:R_Small
- removed U? (x2): 4066, Package_DIP:DIP-14_W7.62mm, symbol 4xxx:4066
- added C11, C12, C13, C14: 10uF, Capacitor_THT:CP_Radial_D4.0mm_P1.50mm, symbol Device:CP1
- added D11, D12: DIODE, Diode_THT:D_T-1_P5.08mm_Horizontal, symbol pspice:DIODE
- added J7, J8: AudioJack3, Connector_Wire:SolderWirePad_1x03_P3.175mm_Drill1mm, symbol Connector:AudioJack3
- added R19, R20, R21, R22, R23, R24, R25, R26: 47K, Resistor_THT:R_Axial_DIN0207_L6.3mm_D2.5mm_P7.62mm_Horizontal, symbol Device:R_Small
- added unit 1 of U4
- added unit 2 of U4
- added unit 3 of U4
- added unit 4 of U4
- C10, C15, C16, C4, C5, C6, C7, C8, C9: renamed from C?; footprint Capacitor_SMD:CP_Elec_3x5.3 -> Capacitor_THT:CP_Radial_D4.0mm_P1.50mm
- C3: renamed from C?; footprint Capacitor_THT:CP_Axial_L10.0mm_D6.0mm_P15.00mm_Horizontal -> Capacitor_THT:CP_Radial_D4.0mm_P1.50mm
- D10, D7, D8, D9: renamed from D?; footprint Diode_SMD:Diode_Bridge_Diotec_ABS -> Diode_THT:D_T-1_P5.08mm_Horizontal
- J3, J4, J5, J6, J9: renamed from J?; footprint Connector_Audio:Jack_3.5mm_CUI_SJ1-3533NG_Horizontal -> Connector_Wire:SolderWirePad_1x03_P3.175mm_Drill1mm
- R10, R11, R12, R13, R14, R15, R16, R17, R18, R3, R4, R5, R6, R7, R8, R9: renamed from R?; footprint Resistor_SMD:R_0201_0603Metric -> Resistor_THT:R_Axial_DIN0207_L6.3mm_D2.5mm_P7.62mm_Horizontal
- gave numbers to parts that had none: 3
Connections:
- net GNDS is gone; now on net GND: J3.S, J4.S, J5.S, J6.S, J9.S
- net GND: now also J7.S, J8.S, R20.2, R22.2, R24.2, R26.2
- net L: now also U4.10, U4.3
- net R: now also U4.2, U4.9
- net VCC: now also R19.1, R21.1, R23.1, R25.1
- net audio_4: now also D12.1 (K), U4.13, U4.5; no longer U4.14 (VDD)
- new net: D11.2 (A), D12.2 (A), U4.14 (VDD)
- new net: C11.1, R19.2, R20.1, U4.1
- new net: C12.1, R21.2, R22.1, U4.4
- new net: C11.2, J7.R
- new net: C12.2, J7.T
- new net: C13.1, R23.2, R24.1, U4.8
- new net: C14.1, R25.2, R26.1, U4.11
- new net: C13.2, J8.R
- new net: C14.2, J8.T
- new net audio_5: D11.1 (K), U4.12, U4.6
Other:
- moved on the sheet: U4E
